File: PCB/Scroll Wheel.kicad_sch (KiCad schematic)
At the start: 39 parts, among them J1 TC2030, J2 USB_C_Receptacle_USB3.1_16P, J3 Conn_01x02_Pin, J4 Conn_01x04_Socket, J5 Conn_01x04_Pin, Q1 FS8205A, Q2 BC847, SW1 SW_Push, U1 ESP32-WROOM-E, U2 BQ25172DSGR, U6 MIC5504-3.3YM5, U7 AS5600

Commit message: fix NMOS to PMOS, and 3d Modells
Parts:
- removed Q1: FS8205A, PCM_Package_TO_SOT_SMD_AKL:SOT-23-6, symbol FS8205A:FS8205A
- removed R30: 1M, Resistor_SMD:R_0402_1005Metric, symbol Device:R
- added Q3: FDC6318P, Package_TO_SOT_SMD:SOT-23-6, symbol PCM_Transistor_MOSFET_AKL:FDC6318P
- added R31: 1M, Resistor_SMD:R_0402_1005Metric, symbol Device:R
- U1: LCSC (none) -> C701342
Connections:
- net BATT: now also Q3.6 (D1)
- net at D5.1 (K), R26.1: now also Q3.1 (G1), Q3.3 (G2), R31.1
- net at C9.2, D3.1 (K), R8.2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: now also Q3.4 (D2)
- new net: Q3.2 (S2), Q3.5 (S1), R31.2
