File: PCB/Scroll Wheel.kicad_sch (KiCad schematic)
At the start: 46 parts, among them J1 TC2030, J2 USB_C_Receptacle_USB3.1_16P, J3 Conn_01x02_Pin, J4 Connector Encoder, J5 Connector controller, Q2 BC847, Q3 FDC6318P, SW1 SW_Push, U1 ESP32-WROOM-E, U2 BQ25172DSGR, U6 MIC5504-3.3YM5, U7 AS5600

Commit message: add a better mounting solution
Parts:
- U2: footprint DSG0008A-IPC_A -> BQ25172:DSG0008A-IPC_A
Changed lines of the file:
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@@
 			)
 		)
-		(property "Footprint" "DSG0008A-IPC_A"
+		(property "Footprint" "BQ25172:DSG0008A-IPC_A"
 			(at 46.99 236.22 0)
 			(effects
